File: Schematics/Artemis Architecture/Artemis ALU.kicad_sch (KiCad schematic)
At the start: 19 parts, among them U1 74LS283, U10 74LS32, U11 74LS86, U12 74LS86, U13 74LS245, U14 74LS245, U15 74LS86, U16 74LS86, U17 74LS08, U18 74LS08, U19 74LS08, U2 74LS283, U3 74LS245, U4 74LS245, U5 74LS245, U6 74LS08, U7 74LS08, U8 74LS245, U9 74LS32

Commit message: Refactored Project Notebook
Parts:
- added U20: 74LS245, Package_DIP:DIP-20_W7.62mm_Socket_LongPads, symbol 74xx:74LS245
- added U21: 74LS32, Package_DIP:DIP-14_W7.62mm_Socket_LongPads, symbol 74xx:74LS32
- added U22: 74LS32, symbol 74xx:74LS32
Connections:
- net at U13.11 (B7), U14.11 (B7), U3.11 (B7)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: now also U20.9 (A7)
- net at U13.12 (B6), U14.12 (B6), U3.12 (B6)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: now also U20.8 (A6)
- net at U13.13 (B5), U14.13 (B5), U3.13 (B5)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: now also U20.7 (A5)
- net at U13.14 (B4), U14.14 (B4), U3.14 (B4)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: now also U20.6 (A4)
- net at U13.15 (B3), U14.15 (B3), U3.15 (B3)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: now also U20.5 (A3)
- net at U13.16 (B2), U14.16 (B2), U3.16 (B2)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: now also U20.4 (A2)
- net at U13.17 (B1), U14.17 (B1), U3.17 (B1)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: now also U20.3 (A1)
- net at U13.18 (B0), U14.18 (B0), U3.18 (B0)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: now also U20.2 (A0)
Other:
- moved on the sheet: U10E, U11E, U12E, U15E, U16E, U17E, U18E, U7E, U9E
