File: Schematics/KICAD Artemis Architecture/_autosave-Artemis ALU.kicad_sch (KiCad schematic)
At the start: 26 parts, among them U1 74LS283, U10 74LS32, U11 74LS86, U12 74LS86, U13 74LS245, U14 74LS245, U15 74LS86, U16 74LS86, U17 74LS08, U18 74LS08, U19 74LS08, U2 74LS283, U20 74LS245, U21 74LS32, U22 74LS32, U23 74LS32, U24 74LS30, U25 74LS30, U26 74LS86, U3 74LS245, U4 74LS245, U5 74LS245, U6 74LS08, U7 74LS08, U8 74LS245, U9 74LS32

Commit message: Removed Carry/Borrow Flag
Parts:
- added U27: 74LS04, symbol 74xx:74LS04
Connections:
- net SU: now also U21.10, U22.2
- net GND: now reaches U13.10 (GND)
- net GND: now also U14.10 (GND), U20.10 (GND), U3.10 (GND), U4.10 (GND), U5.10 (GND), U8.10 (GND)
- net at U26.6: no longer U20.19 (CE)
- net at U3.19 (CE): now also U27.2
- net AD: now reaches U21.9
- net AD: now also U22.1
- net at U23.3: now also U27.1
- net EN: no longer names the net of U26.5
- net VCC: no longer names the net of U26.4
- new net ~EN: U20.19 (CE)
Other:
- moved on the sheet: U21C, U21D, U23A, U26B
