File: Schematics/KICAD Artemis Architecture/Artemis ALU.kicad_sch (KiCad schematic)
At the start: 22 parts, among them U1 74LS283, U10 74LS32, U11 74LS86, U12 74LS86, U13 74LS245, U14 74LS245, U15 74LS86, U16 74LS86, U17 74LS08, U18 74LS08, U19 74LS08, U2 74LS283, U20 74LS245, U21 74LS32, U22 74LS32, U3 74LS245, U4 74LS245, U5 74LS245, U6 74LS08, U7 74LS08, U8 74LS245, U9 74LS32

Commit message: ALU Updates
Parts:
- added U23: 74LS32, Package_DIP:DIP-14_W7.62mm_Socket_LongPads, symbol 74xx:74LS32
- added U24, U25: 74LS30, symbol 74xx:74LS30
- added U26: 74LS86, Package_DIP:DIP-14_W7.62mm_Socket_LongPads, symbol 74xx:74LS86
Connections:
- net at U15.10, U15.13, U15.2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: now also U21.3
- net at U13.11 (B7), U14.11 (B7), U20.9 (A7)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: now also U25.12
- net at U13.12 (B6), U14.12 (B6), U20.8 (A6)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: now also U25.11
- net at U13.13 (B5), U14.13 (B5), U20.7 (A5)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: now also U25.6
- net at U13.14 (B4), U14.14 (B4), U20.6 (A4)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: now also U25.5
- net at U13.15 (B3), U14.15 (B3), U20.5 (A3)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: now also U25.4
- net at U13.16 (B2), U14.16 (B2), U20.4 (A2)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: now also U25.3
- net at U13.17 (B1), U14.17 (B1), U20.3 (A1)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: now also U25.2
- net at U13.18 (B0), U14.18 (B0), U20.2 (A0)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: now also U25.1
- net at U1.9 (C4): now also U26.2
- net at U17.10, U17.13, U18.10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: now also U22.11
- net at U2.7 (C0): now also U21.6
- net at U21.11: now also U23.2
- net at U22.6: now also U22.10
- net at U22.12: now also U22.8
- net at U22.9: now also U22.3
- net EN: now reaches U20.19 (CE)
- net at U21.8: now also U23.1
- new net: U23.6, U26.1
Other:
- moved on the sheet: U10E, U11E, U12E, U15E, U16E, U17E, U18E, U21A, U21B, U21C, U21D, U21E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

Commit message: Removed Carry/Borrow Flag
Connections:
- net EN: now also U26.5; no longer U20.19 (CE)
- net GND: now reaches U13.10 (GND)
- net GND: now also U14.10 (GND), U20.10 (GND), U3.10 (GND), U4.10 (GND), U5.10 (GND), U8.10 (GND)
- net VCC: now reaches U26.4
- net at U26.6: now also U20.19 (CE)
Other:
- moved on the sheet: U26B

Commit message: Replaced custom ALU with the 74ls181
Parts:
- removed unit 2 of U23
- removed unit 1 of U26
- added R1, R2, R3, R4, R5, R6, R7, R8: 10k, Resistor_SMD:R_1206_3216Metric_Pad1.30x1.75mm_HandSolder, symbol Device:R
- added U27: 74LS04, symbol 74xx:74LS04
Connections:
- net DC: now also U21.13, U21.2
- net GND: now also U1.8 (GND), U10.7 (GND), U11.7 (GND), U12.7 (GND), U15.7 (GND), U16.7 (GND), U17.7 (GND), U18.7 (GND), U2.8 (GND), U21.7 (GND), U22.7 (GND), U23.7 (GND), U24.7 (GND), U26.7 (GND), U6.7 (GND), U7.7 (GND), U9.7 (GND), U27.7 (GND)
- net IC: now also U21.12, U21.5
- net SU: now also U21.1, U21.10, U21.4, U22.2
- net VCC: now also U1.16 (VCC), U10.14 (VCC), U11.14 (VCC), U12.14 (VCC), U13.20 (VCC), U14.20 (VCC), U15.14 (VCC), U16.14 (VCC), U17.14 (VCC), U18.14 (VCC), U2.16 (VCC), U20.20 (VCC), U21.14 (VCC), U22.14 (VCC), U23.14 (VCC), U24.14 (VCC), U26.14 (VCC), U3.20 (VCC), U4.20 (VCC), U5.20 (VCC), U6.14 (VCC), U7.14 (VCC), U8.20 (VCC), U9.14 (VCC), R1.2, R2.2, R3.2, R4.2, R5.2, R6.2, R7.2, R8.2, U27.14 (VCC); no longer U26.4
- net at U13.11 (B7), U14.11 (B7), U20.9 (A7)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: now also R8.1
- net at U13.12 (B6), U14.12 (B6), U20.8 (A6)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: now also R7.1
- net at U13.13 (B5), U14.13 (B5), U20.7 (A5)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: now also R6.1
- net at U13.14 (B4), U14.14 (B4), U20.6 (A4)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: now also R5.1
- net at U13.15 (B3), U14.15 (B3), U20.5 (A3)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: now also R4.1
- net at U13.16 (B2), U14.16 (B2), U20.4 (A2)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: now also R3.1
- net at U13.17 (B1), U14.17 (B1), U20.3 (A1)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: now also R2.1
- net at U13.18 (B0), U14.18 (B0), U20.2 (A0)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: now also R1.1
- net at U13.19 (CE): now also U27.6
- net at U26.6: no longer U20.19 (CE)
- net at U3.19 (CE): now also U27.2
- net at U5.19 (CE): now also U27.10
- net at U14.19 (CE): now also U27.8
- net at U8.19 (CE): now also U27.4
- net AN: now reaches U22.4
- net AN: now also U27.3
- net OR: now reaches U22.5
- net OR: now also U27.5
- net XO: now reaches U22.13
- net XO: now also U27.9
- net ALU 5: now reaches U20.13 (B5)
- net ALU 4: now reaches U20.14 (B4)
- net ALU 3: now reaches U20.15 (B3)
- net ALU 2: now reaches U20.16 (B2)
- net ALU 1: now reaches U20.17 (B1)
- net ALU 0: now reaches U20.18 (B0)
- net AD: now reaches U21.9
- net AD: now also U22.1
- net at U23.3: now also U27.1
- net at U4.19 (CE): now also U27.12
- net EN: no longer names the net of U26.5
- new net RL: U27.13
- new net RR: U27.11
- new net ~EN: U20.19 (CE)
Other:
- moved on the sheet: U10E, U11E, U12E, U15E, U16E, U17E, U18E, U21B, U21C, U21D, U21E, U22E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
