File: Schematics/KICAD Artemis Architecture/DEPRICATED Custom ALU/Artemis ALU.kicad_sch (KiCad schematic)
At the start: 27 parts, among them U1 74LS283, U10 74LS32, U11 74LS86, U12 74LS86, U13 74LS245, U14 74LS245, U15 74LS86, U16 74LS86, U17 74LS08, U18 74LS08, U19 74LS08, U2 74LS283, U20 74LS245, U21 74LS32, U22 74LS32, U23 74LS32, U24 74LS30, U25 74LS30, U26 74LS86, U27 74LS04, U3 74LS245, U4 74LS245, U5 74LS245, U6 74LS08, U7 74LS08, U8 74LS245, U9 74LS32

Commit message: Replaced custom ALU with the 74ls181
Parts:
- removed unit 2 of U23
- removed unit 1 of U26
- added R1, R2, R3, R4, R5, R6, R7, R8: 10k, Resistor_SMD:R_1206_3216Metric_Pad1.30x1.75mm_HandSolder, symbol Device:R
Connections:
- net AN: now also U22.4, U27.3
- net DC: now also U21.13, U21.2
- net GND: now also U1.8 (GND), U10.7 (GND), U11.7 (GND), U12.7 (GND), U15.7 (GND), U16.7 (GND), U17.7 (GND), U18.7 (GND), U2.8 (GND), U21.7 (GND), U22.7 (GND), U23.7 (GND), U24.7 (GND), U26.7 (GND), U27.7 (GND), U6.7 (GND), U7.7 (GND), U9.7 (GND)
- net IC: now also U21.12, U21.5
- net OR: now also U22.5, U27.5
- net RL: now also U27.13
- net RR: now also U27.11
- net SU: now also U21.1, U21.4
- net XO: now also U22.13, U27.9
- net at U13.11 (B7), U14.11 (B7), U20.9 (A7)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: now also R8.1
- net at U13.12 (B6), U14.12 (B6), U20.8 (A6)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: now also R7.1
- net at U13.13 (B5), U14.13 (B5), U20.7 (A5)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: now also R6.1
- net at U13.14 (B4), U14.14 (B4), U20.6 (A4)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: now also R5.1
- net at U13.15 (B3), U14.15 (B3), U20.5 (A3)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: now also R4.1
- net at U13.16 (B2), U14.16 (B2), U20.4 (A2)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: now also R3.1
- net at U13.17 (B1), U14.17 (B1), U20.3 (A1)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: now also R2.1
- net at U13.18 (B0), U14.18 (B0), U20.2 (A0)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: now also R1.1
- net at U13.19 (CE): now also U27.6
- net VCC: now reaches U13.20 (VCC)
- net VCC: now also U1.16 (VCC), U10.14 (VCC), U11.14 (VCC), U12.14 (VCC), U14.20 (VCC), U15.14 (VCC), U16.14 (VCC), U17.14 (VCC), U18.14 (VCC), U2.16 (VCC), U20.20 (VCC), U21.14 (VCC), U22.14 (VCC), U23.14 (VCC), U24.14 (VCC), U26.14 (VCC), U27.14 (VCC), U3.20 (VCC), U4.20 (VCC), U5.20 (VCC), U6.14 (VCC), U7.14 (VCC), U8.20 (VCC), U9.14 (VCC), R1.2, R2.2, R3.2, R4.2, R5.2, R6.2, R7.2, R8.2
- net at U27.4: now also U8.19 (CE)
- net at U5.19 (CE): now also U27.10
- net at U14.19 (CE): now also U27.8
- net ALU 5: now reaches U20.13 (B5)
- net ALU 4: now reaches U20.14 (B4)
- net ALU 3: now reaches U20.15 (B3)
- net ALU 2: now reaches U20.16 (B2)
- net ALU 1: now reaches U20.17 (B1)
- net ALU 0: now reaches U20.18 (B0)
- net at U4.19 (CE): now also U27.12
Other:
- moved on the sheet: U10E, U11E, U12E, U15E, U16E, U17E, U18E, U21B, U21E, U22E, U23E, U24B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
