File: Schematics/KICAD Artemis Architecture/Artemis ALU/Artemis ALU Module.kicad_pcb (KiCad board)
At the start: 4 copper layers, 66.2 x 46 mm, 11 parts, among them J1 B Input Socket, J2 A Input Socket, J3 F Output Socket, J4 Control Word Socket, J5 Flag Socket, J6 Power Socket, U1 74LS181, U2 74LS181, U3 74LS30

Commit message: Completed ALU PCB
Other:
- board text added: "74LS30"
- board text added: "A Input"
- board text added: "ALU Module"
- board text added: "B Input"
- board text added: "Control"
- board text added: "Flags"
- board text added: "George Sleen"
- board text added: "Output"
- board text added: "Power"
