File: Schematics/KICAD Artemis Architecture/Instruction register/Instruction register.kicad_sch (KiCad schematic)
At the start: 44 parts, among them J1 Power, J2 Control, J3 BUS LB, J4 BUS UB, J5 Instruction Out, U1 74LS173, U2 74LS245, U3 74LS173, U4 74LS173, U5 74LS173, U6 74LS245

Commit message: Instruction Register Complete
Parts:
- added C2: 0.1 uF, Capacitor_SMD:C_1206_3216Metric_Pad1.33x1.80mm_HandSolder, symbol Device:C
Connections:
- net CLR: now also C2.1
- net GNDREF: now also C2.2
Changed lines of the file:
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@@
 	)
 	(junction
+		(at 97.79 237.49)
+		(diameter 0)
+		(color 0 0 0 0)
+	)
+	(junction
 		(at 115.57 238.76)
 		(diameter 0)
@@
 	(wire
 		(pts
-			(xy 58.42 237.49) (xy 231.14 237.49)
+			(xy 58.42 237.49) (xy 97.79 237.49)
 		)
 		(stroke
@@
 	(wire
 		(pts
+			(xy 97.79 237.49) (xy 231.14 237.49)
+		)
+		(stroke
+			(width 0)
+			(type default)
+		)
+	)
+	(wire
+		(pts
 			(xy 231.14 166.37) (xy 231.14 237.49)
 		)
@@
 	(wire
 		(pts
+			(xy 97.79 237.49) (xy 97.79 259.08)
+		)
+		(stroke
+			(width 0)
+			(type default)
+		)
+	)
+	(wire
+		(pts
 			(xy 44.45 236.22) (xy 57.15 236.22)
 		)
@@
 		)
 	)
+	(text_box "RST Decoupling Capacitor"
+		(exclude_from_sim no)
+		(at 92.71 256.54 0)
+		(size 19.05 17.78)
+		(stroke
+			(width 0)
+			(type default)
+		)
+		(fill
+			(type none)
+		)
+		(effects
+			(font
+				(size 1.27 1.27)
+			)
+			(justify left top)
+		)
+	)
 	(text_box "UB"
 		(exclude_from_sim no)
@@
 	)
 	(symbol
+		(lib_id "power:GNDREF")
+		(at 97.79 266.7 0)
+		(unit 1)
+		(exclude_from_sim no)
+		(in_bom yes)
+		(on_board yes)
+		(dnp no)
+		(fields_autoplaced yes)
+		(property "Reference" "#PWR023"
+			(at 97.79 273.05 0)
+			(effects
+				(font
+					(size 1.27 1.27)
+				)
+				(hide yes)
+			)
+		)
+		(property "Value" "GNDREF"
+			(at 97.79 271.78 0)
+			(effects
+				(font
+					(size 1.27 1.27)
+				)
+			)
+		)
+		(property "Footprint" ""
+			(at 97.79 266.7 0)
+			(effects
+				(font
+					(size 1.27 1.27)
+				)
+				(hide yes)
+			)
+		)
+		(property "Datasheet" ""
+			(at 97.79 266.7 0)
+			(effects
+				(font
+					(size 1.27 1.27)
+				)
+				(hide yes)
+			)
+		)
+		(property "Description" "Power symbol creates a global label with name \"GNDREF\" , reference supply ground"
+			(at 97.79 266.7 0)
+			(effects
+				(font
+					(size 1.27 1.27)
+				)
+				(hide yes)
+			)
+		)
+		(pin "1"
+		)
+		(instances
+			(project "Instruction register"
+				(path "/f964096b-9e13-43c1-bf2d-ba0caa73513f"
+					(reference "#PWR023")
+					(unit 1)
+				)
+			)
+		)
+	)
+	(symbol
 		(lib_id "Device:LED")
 		(at 307.34 158.75 90)
@@
 					(unit 1)
 				)
+			)
+		)
+	)
+	(symbol
+		(lib_id "Device:C")
+		(at 97.79 262.89 0)
+		(unit 1)
+		(exclude_from_sim no)
+		(in_bom yes)
+		(on_board yes)
+		(dnp no)
+		(fields_autoplaced yes)
+		(property "Reference" "C2"
+			(at 101.6 261.6199 0)
+			(effects
+				(font
+					(size 1.27 1.27)
+				)
+				(justify left)
+			)
+		)
+		(property "Value" "0.1 uF"
+			(at 101.6 264.1599 0)
+			(effects
+				(font
+					(size 1.27 1.27)
+				)
+				(justify left)
+			)
+		)
+		(property "Footprint" "Capacitor_SMD:C_1206_3216Metric_Pad1.33x1.80mm_HandSolder"
+			(at 98.7552 266.7 0)
+			(effects
+				(font
+					(size 1.27 1.27)
+				)
+				(hide yes)
+			)
+		)
+		(property "Datasheet" "~"
+			(at 97.79 262.89 0)
+			(effects
+				(font
+					(size 1.27 1.27)
+				)
+				(hide yes)
+			)
+		)
+		(property "Description" "Unpolarized capacitor"
+			(at 97.79 262.89 0)
+			(effects
+				(font
+					(size 1.27 1.27)
+				)
+				(hide yes)
+			)
+		)
+		(pin "1"
+		)
+		(pin "2"
+		)
+		(instances
+			(project "Instruction register"
+				(path "/f964096b-9e13-43c1-bf2d-ba0caa73513f"
+					(reference "C2")
+					(unit 1)
+				)
