File: Schematics/KICAD Artemis Architecture/Control Logic/Control Logic V1.kicad_sch (KiCad schematic)
At the start: 5 parts, among them IC1 AT28C64B-15PU, IC2 AT28C64B-15PU, IC3 AT28C64B-15PU, J1 Instruction, J2 Flags

Commit message: whatever
Parts:
- added D1, D2, D3: LED, LED_SMD:LED_1206_3216Metric_Pad1.42x1.75mm_HandSolder, symbol Device:LED
- added R1, R2, R3: 220, Resistor_SMD:R_1206_3216Metric_Pad1.30x1.75mm_HandSolder, symbol Device:R
- added U1: 74LS161, Package_DIP:DIP-16_W7.62mm_Socket_LongPads, symbol 74xx:74LS161
- added U2, U3: 74LS138, Package_DIP:DIP-16_W7.62mm_Socket_LongPads, symbol 74xx:74LS138
- added U4: 74LS02, Package_DIP:DIP-14_W7.62mm_Socket_LongPads, symbol 74xx:74LS02
Connections:
- net GNDREF: now also IC1.20 (~{CE}), IC1.22 (~{OE}), IC2.20 (~{CE}), IC2.22 (~{OE}), IC3.20 (~{CE}), IC3.22 (~{OE}), R1.2, R2.2, R3.2, U1.3 (D0), U1.4 (D1), U1.5 (D2), U1.6 (D3), U1.8 (GND)
- net Microcode early exit: now also U4.2
- net VCC: now also IC1.27 (~{WE}), IC2.27 (~{WE}), IC3.27 (~{WE}), U1.10 (CET), U1.16 (VCC), U1.7 (CEP), U1.9 (~{PE})
- net at IC2.2 (A12): now also IC1.2 (A12), IC3.2 (A12), J2.2 (Pin_2)
- net at IC2.21 (A10): now also IC1.21 (A10), IC3.21 (A10), D3.2 (A), U1.12 (Q2)
- net at IC2.23 (A11): now also IC1.23 (A11), IC3.23 (A11), J2.1 (Pin_1)
- net at IC2.24 (A9): now also IC1.24 (A9), IC3.24 (A9), D2.2 (A), U1.13 (Q1)
- net at IC2.25 (A8): now also IC1.25 (A8), IC3.25 (A8), D1.2 (A), U1.14 (Q0)
- new net: D3.1 (K), R3.1
- new net: D2.1 (K), R2.1
- new net: D1.1 (K), R1.1
- new net: U1.1 (~{MR}), U4.1
- no-connect marks 3 -> 8
